Commit message: modified maxTorque from 10 to 50 Nm

File: data/Full_robot_urdf/urdf/Full_robot_urdf.urdf (robot description, URDF)
Before this commit: robot Full_robot_urdf, 13 links, 12 joints
Joints:
- joint Knee1_joint: limit lower=1.05 upper=4.54 effort=10 velocity=4 -> lower=1.05 upper=4.54 effort=50 velocity=4
- joint Knee2_joint: limit lower=1.05 upper=4.54 effort=10 velocity=4 -> lower=1.05 upper=4.54 effort=50 velocity=4
- joint Knee3_joint: limit lower=1.05 upper=4.54 effort=10 velocity=4 -> lower=1.05 upper=4.54 effort=50 velocity=4
- joint Knee4_joint: limit lower=1.05 upper=4.54 effort=10 velocity=4 -> lower=1.05 upper=4.54 effort=50 velocity=4
- joint Shoulder1_joint: limit lower=2.09 upper=3.66 effort=10 velocity=4 -> lower=2.09 upper=3.66 effort=50 velocity=4
- joint Shoulder2_joint: limit lower=2.09 upper=3.66 effort=10 velocity=4 -> lower=2.09 upper=3.66 effort=50 velocity=4
- joint Shoulder3_joint: limit lower=2.09 upper=3.66 effort=10 velocity=4 -> lower=2.09 upper=3.66 effort=50 velocity=4
- joint Shoulder4_joint: limit lower=2.09 upper=3.66 effort=10 velocity=4 -> lower=2.09 upper=3.66 effort=50 velocity=4
- joint Waist1_joint: limit lower=0 upper=1.22 effort=10 velocity=4 -> lower=0 upper=1.22 effort=50 velocity=4
- joint Waist2_joint: limit lower=0 upper=1.22 effort=10 velocity=4 -> lower=0 upper=1.22 effort=50 velocity=4
- joint Waist3_joint: limit lower=0 upper=1.22 effort=10 velocity=4 -> lower=0 upper=1.22 effort=50 velocity=4
- joint Waist4_link: limit lower=0 upper=1.22 effort=10 velocity=4 -> lower=0 upper=1.22 effort=50 velocity=4

Commit message: fixed coordinate systems in urdf

File: data/Full_robot_urdf/urdf/Full_robot_urdf.urdf (robot description, URDF)
Before this commit: robot Full_robot_urdf, 13 links, 12 joints
Joints:
- joint Knee1_joint: limit lower=1.05 upper=4.54 effort=50 velocity=4 -> lower=-0.60 upper=2.30 effort=50 velocity=4
- joint Knee2_joint: limit lower=1.05 upper=4.54 effort=50 velocity=4 -> lower=-0.60 upper=2.30 effort=50 velocity=4
- joint Knee3_joint: limit lower=1.05 upper=4.54 effort=50 velocity=4 -> lower=-0.60 upper=2.30 effort=50 velocity=4
- joint Knee4_joint: limit lower=1.05 upper=4.54 effort=50 velocity=4 -> lower=-0.60 upper=2.30 effort=50 velocity=4
- joint Shoulder1_joint: axis 0 0 -1 -> 0 0 1; limit lower=2.09 upper=3.66 effort=50 velocity=4 -> lower=-0.75 upper=0.75 effort=50 velocity=4
- joint Shoulder2_joint: limit lower=2.09 upper=3.66 effort=50 velocity=4 -> lower=-0.75 upper=0.75 effort=50 velocity=4
- joint Shoulder3_joint: limit lower=2.09 upper=3.66 effort=50 velocity=4 -> lower=-0.75 upper=0.75 effort=50 velocity=4
- joint Shoulder4_joint: axis 0 0 -1 -> 0 0 1; limit lower=2.09 upper=3.66 effort=50 velocity=4 -> lower=-0.75 upper=0.75 effort=50 velocity=4
- joint Waist1_joint: limit lower=0 upper=1.22 effort=50 velocity=4 -> lower=0 upper=0.90 effort=50 velocity=4
- joint Waist2_joint: limit lower=0 upper=1.22 effort=50 velocity=4 -> lower=0 upper=0.90 effort=50 velocity=4
- joint Waist3_joint: limit lower=0 upper=1.22 effort=50 velocity=4 -> lower=0 upper=0.90 effort=50 velocity=4
- joint Waist4_link: limit lower=0 upper=1.22 effort=50 velocity=4 -> lower=0 upper=0.90 effort=50 velocity=4

Commit message: somehwat working gait

File: data/Full_robot_urdf/urdf/Full_robot_urdf.urdf (robot description, URDF)
Before this commit: robot Full_robot_urdf, 13 links, 12 joints
Links:
- added link Foot1_link, mass 0.05; collision sphere radius=0.02; visual sphere radius=0.02
- added link Foot2_link, mass 0.05; collision sphere radius=0.02; visual sphere radius=0.02
- added link Foot3_link, mass 0.05; collision sphere radius=0.02; visual sphere radius=0.02
- added link Foot4_link, mass 0.05; collision sphere radius=0.02; visual sphere radius=0.02
- link base_link: mass 26.5470635630031 -> 10.5470635630031
Joints:
- added joint Foot1_joint: type fixed, parent Knee1_link, child Foot1_link, origin xyz=0 0.1019 0 rpy=0 0 0
- added joint Foot2_joint: type fixed, parent Knee2_link, child Foot2_link, origin xyz=0 0.1019 0 rpy=0 0 0
- added joint Foot3_joint: type fixed, parent Knee3_link, child Foot3_link, origin xyz=0 0.1019 0 rpy=0 0 0
- added joint Foot4_joint: type fixed, parent Knee4_link, child Foot4_link, origin xyz=0 0.1019 0 rpy=0 0 0
- joint Knee1_joint: limit lower=-0.60 upper=2.30 effort=50 velocity=4 -> lower=-0.60 upper=2.30 effort=100 velocity=4
- joint Knee2_joint: limit lower=-0.60 upper=2.30 effort=50 velocity=4 -> lower=-0.60 upper=2.30 effort=100 velocity=4
- joint Knee3_joint: limit lower=-0.60 upper=2.30 effort=50 velocity=4 -> lower=-0.60 upper=2.30 effort=100 velocity=4
- joint Knee4_joint: limit lower=-0.60 upper=2.30 effort=50 velocity=4 -> lower=-0.60 upper=2.30 effort=100 velocity=4
- joint Shoulder1_joint: limit lower=-0.75 upper=0.75 effort=50 velocity=4 -> lower=-0.75 upper=0.75 effort=100 velocity=4
- joint Shoulder2_joint: limit lower=-0.75 upper=0.75 effort=50 velocity=4 -> lower=-0.75 upper=0.75 effort=100 velocity=4
- joint Shoulder3_joint: limit lower=-0.75 upper=0.75 effort=50 velocity=4 -> lower=-0.75 upper=0.75 effort=100 velocity=4
- joint Shoulder4_joint: limit lower=-0.75 upper=0.75 effort=50 velocity=4 -> lower=-0.75 upper=0.75 effort=100 velocity=4
- joint Waist1_joint: limit lower=0 upper=0.90 effort=50 velocity=4 -> lower=0 upper=0.90 effort=100 velocity=4
- joint Waist2_joint: limit lower=0 upper=0.90 effort=50 velocity=4 -> lower=0 upper=0.90 effort=100 velocity=4
- joint Waist3_joint: limit lower=0 upper=0.90 effort=50 velocity=4 -> lower=0 upper=0.90 effort=100 velocity=4
- joint Waist4_link: limit lower=0 upper=0.90 effort=50 velocity=4 -> lower=0 upper=0.90 effort=100 velocity=4

Commit message: idk...added sliders and limited elbow joints

File: data/Full_robot_urdf/urdf/Full_robot_urdf.urdf (robot description, URDF)
Before this commit: robot Full_robot_urdf, 17 links, 16 joints
Joints:
- joint Knee1_joint: limit lower=-0.60 upper=2.30 effort=100 velocity=4 -> lower=-0.60 upper=1.0 effort=100 velocity=4
- joint Knee2_joint: limit lower=-0.60 upper=2.30 effort=100 velocity=4 -> lower=-0.60 upper=1.0 effort=100 velocity=4
- joint Knee3_joint: limit lower=-0.60 upper=2.30 effort=100 velocity=4 -> lower=-0.60 upper=1.0 effort=100 velocity=4
- joint Knee4_joint: limit lower=-0.60 upper=2.30 effort=100 velocity=4 -> lower=-0.60 upper=1.0 effort=100 velocity=4
